Commit message: setup nav on dev machine

File: mini_description/urdf/body/mini_chassis.urdf.xacro (robot description, xacro)
@@ -13,5 +13,5 @@
             </geometry> -->
             <geometry>
-                <mesh filename="package://mini_description/meshes/Chassis.stl" scale="1 1 1"/>
+                <mesh filename="package://mini_description/meshes/shifted_base.stl" scale="0.001 0.001 0.001"/>
             </geometry>
             <origin xyz="0.0 0.0 0.0" rpy="0.0 0.0 0.0"/>
@@ -20,5 +20,5 @@
         <collision>
             <geometry>
-                <box size="${base_length} ${base_width} ${base_height}"/>
+                <mesh filename="package://mini_description/meshes/shifted_base.stl" scale="0.001 0.001 0.001"/>
             </geometry>
             <origin xyz="0 0 ${base_height/2}" rpy="0 0 0"/>
@@ -35,5 +35,5 @@
         <origin xyz="0.0 0.0 0.0235" rpy="0.0 0.0 0.0"/>
         <parent link="base_footprint"/>
-        <child link="base_link"/>
+        <child link="${prefix}base_link"/>
     </joint>
 </xacro:macro>

File: mini_description/urdf/body/mini_robot.urdf.xacro (robot description, xacro)
@@ -17,20 +17,40 @@
     <xacro:mini_chassis
     prefix="$(arg prefix)" />
-    <xacro:mini_wheels
+    <xacro:front_wheel_rods
+            prefix="$(arg prefix)"
+            side="front_right_wheel_rod"
+            x_reflect="1"
+            y_reflect="-1"/>
+    <xacro:front_wheel_rods
+            prefix="$(arg prefix)"
+            side="front_left_wheel_rod"
+            x_reflect="1"
+            y_reflect="1"/>
+    <xacro:rear_wheel_rods
         prefix="$(arg prefix)"
-        side="front_right_wheel"
-        x_reflect="1"
+        side="rear_left_wheel_rod"
+        x_reflect="-1"
+        y_reflect="1"/>
+    <xacro:rear_wheel_rods
+        prefix="$(arg prefix)"
+        side="rear_right_wheel_rod"
+        x_reflect="-1"
         y_reflect="-1"/>
-    <xacro:mini_wheels
+    <xacro:front_mini_wheels
+            prefix="$(arg prefix)"
+            side="front_right_wheel"
+            x_reflect="1"
+            y_reflect="-1"/>
+    <xacro:front_mini_wheels
         prefix="$(arg prefix)"
         side="front_left_wheel"
         x_reflect="1"
         y_reflect="1"/>
-    <xacro:mini_wheels
+    <xacro:rear_mini_wheels
         prefix="$(arg prefix)"
         side="rear_left_wheel"
         x_reflect="-1"
         y_reflect="1"/>
-    <xacro:mini_wheels
+    <xacro:rear_mini_wheels
         prefix="$(arg prefix)"
         side="rear_right_wheel"

File: mini_description/urdf/body/mini_wheels.urdf.xacro (robot description, xacro)
@@ -1,11 +1,85 @@
 <?xml version="1.0"?>
 <robot xmlns:xacro="http://www.ros.org/wiki/xacro">
+    <xacro:property name="rod_radius" value="0.0025" />
+    <xacro:property name="rod_width" value="0.012" />
+    <xacro:property name="rod_xoff" value="0.061" />
+    <xacro:property name="rod_yoff" value="0.077" />
+    <xacro:property name="rod_zoff" value="-0.017003" />
+    <xacro:property name="rear_rod_xoff" value="0.050" />
+    <xacro:property name="rear_rod_yoff" value="0.077" />
     <xacro:property name="wheel_radius" value="0.022" />
     <xacro:property name="wheel_width" value="0.02" />
-    <xacro:property name="wheel_mass" value="0.04" />
-    <xacro:property name="wheel_xoff" value="0.076123" />
-    <xacro:property name="wheel_yoff" value="0.1010" />
+    <xacro:property name="wheel_mass" value="0.4" />
+    <xacro:property name="wheel_yoff" value="${wheel_width/2}" />
+    <!-- <xacro:property name="wheel_xoff" value="0.061" />
+    <xacro:property name="wheel_yoff" value="0.087" />
     <xacro:property name="wheel_zoff" value="-0.017003" />
-    <xacro:macro name="mini_wheels" params="prefix side x_reflect y_reflect">
+    <xacro:property name="rear_wheel_xoff" value="0.050" />
+    <xacro:property name="rear_wheel_yoff" value="0.087" /> -->
+    <xacro:macro name="front_wheel_rods" params="prefix side x_reflect y_reflect">
+        <link name="${prefix}${side}_link">
+            <visual>
+                <origin xyz="0.0 0.0 0.0" rpy="${pi/2} 0.0 0.0"/>
+                <geometry>
+                    <cylinder radius="${rod_radius}" length="${rod_width}"/>
+                </geometry>
+                <material name="black">
+                        <color rgba="0.5 0.5 0.5 0.5"/>
+                </material>
+            </visual>
+            <collision>
+                <origin xyz="0 0 0" rpy="${pi/2} 0 0"/>
+                <geometry>
+                    <cylinder radius="${rod_radius}" length="${rod_width}"/>
+                </geometry>
+            </collision>
+            <inertial>
+                <origin xyz="0 0 0" rpy="0 0 0"/>
+                <mass value="${wheel_mass}"/>
+                <inertia
+                ixx="${(wheel_mass/12.0) * (3*wheel_radius*wheel_radius + wheel_width*wheel_width)}" ixy="0" ixz="0"
+                iyy="${(wheel_mass/2.0) * (wheel_radius*wheel_radius)}" iyz="0"
+                izz="${(wheel_mass/12.0) * (3*wheel_radius*wheel_radius + wheel_width*wheel_width)}"/>
+            </inertial>
+        </link>
+        <joint name="${side}_joint" type="fixed">
+            <origin xyz="${x_reflect*rod_xoff} ${y_reflect*rod_yoff} ${rod_zoff}" rpy="0.0 0.0 0.0"/>
+            <parent link="${prefix}base_link"/>
+            <child link="${prefix}${side}_link"/>
+        </joint>
+    </xacro:macro>
+    <xacro:macro name="rear_wheel_rods" params="prefix side x_reflect y_reflect">
+        <link name="${prefix}${side}_link">
+            <visual>
+                <origin xyz="0.0 0.0 0.0" rpy="${pi/2} 0.0 0.0"/>
+                <geometry>
+                    <cylinder radius="${rod_radius}" length="${rod_width}"/>
+                </geometry>
+                <material name="black">
+                        <color rgba="0.5 0.5 0.5 0.5"/>
+                </material>
+            </visual>
+            <collision>
+                <origin xyz="0 0 0" rpy="${pi/2} 0 0"/>
+                <geometry>
+                    <cylinder radius="${rod_radius}" length="${rod_width}"/>
+                </geometry>
+            </collision>
+            <inertial>
+                <origin xyz="0 0 0" rpy="0 0 0"/>
+                <mass value="${wheel_mass}"/>
+                <inertia
+                ixx="${(wheel_mass/12.0) * (3*wheel_radius*wheel_radius + wheel_width*wheel_width)}" ixy="0" ixz="0"
+                iyy="${(wheel_mass/2.0) * (wheel_radius*wheel_radius)}" iyz="0"
+                izz="${(wheel_mass/12.0) * (3*wheel_radius*wheel_radius + wheel_width*wheel_width)}"/>
+            </inertial>
+        </link>
+        <joint name="${side}_joint" type="fixed">
+            <origin xyz="${x_reflect*rear_rod_xoff} ${y_reflect*rear_rod_yoff} ${rod_zoff}" rpy="0.0 0.0 0.0"/>
+            <parent link="${prefix}base_link"/>
+            <child link="${prefix}${side}_link"/>
+        </joint>
+    </xacro:macro>
+    <xacro:macro name="front_mini_wheels" params="prefix side x_reflect y_reflect">
         <link name="${prefix}${side}_link">
             <visual>
@@ -14,6 +88,6 @@
                     <cylinder radius="${wheel_radius}" length="${wheel_width}"/>
                 </geometry>
-                <material name="black">
-                        <color rgba="0.0 0.0 0.0 1.0"/>
+                <material name="grey">
+                        <color rgba="0.5 0.5 0.5 0.5"/>
                 </material>
             </visual>
@@ -34,7 +108,40 @@
         </link>
         <joint name="${side}_joint" type="continuous">
-            <origin xyz="${x_reflect*wheel_xoff} ${y_reflect*wheel_yoff} ${wheel_zoff}" rpy="0.0 0.0 0.0"/>
-            <parent link="base_link"/>
-            <child link="${side}_link"/>
+            <origin xyz="0 ${y_reflect*wheel_yoff} 0" rpy="0.0 0.0 0.0"/>
+            <parent link="${prefix}${side}_rod_link"/>
+            <child link="${prefix}${side}_link"/>
+            <axis xyz="0.0 1.0 0.0"/>
+        </joint>
+    </xacro:macro>
+    <xacro:macro name="rear_mini_wheels" params="prefix side x_reflect y_reflect">
+        <link name="${prefix}${side}_link">
+            <visual>
+                <origin xyz="0.0 0.0 0.0" rpy="${pi/2} 0.0 0.0"/>
+                <geometry>
+                    <cylinder radius="${wheel_radius}" length="${wheel_width}"/>
+                </geometry>
+                <material name="grey">
+                        <color rgba="0.5 0.5 0.5 0.5"/>
+                </material>
+            </visual>
+            <collision>
+                <origin xyz="0 0 0" rpy="${pi/2} 0 0"/>
+                <geometry>
+                    <cylinder radius="${wheel_radius}" length="${wheel_width}"/>
+                </geometry>
+            </collision>
+            <inertial>
+                <origin xyz="0 0 0" rpy="0 0 0"/>
+                <mass value="${wheel_mass}"/>
+                <inertia
+                ixx="${(wheel_mass/12.0) * (3*wheel_radius*wheel_radius + wheel_width*wheel_width)}" ixy="0" ixz="0"
+                iyy="${(wheel_mass/2.0) * (wheel_radius*wheel_radius)}" iyz="0"
+                izz="${(wheel_mass/12.0) * (3*wheel_radius*wheel_radius + wheel_width*wheel_width)}"/>
+            </inertial>
+        </link>
+        <joint name="${side}_joint" type="continuous">
+            <origin xyz="0 ${y_reflect*wheel_yoff} 0" rpy="0.0 0.0 0.0"/>
+            <parent link="${prefix}${side}_rod_link"/>
+            <child link="${prefix}${side}_link"/>
             <axis xyz="0.0 1.0 0.0"/>
         </joint>

File: mini_description/urdf/gazebo/mini_gazebo.urdf.xacro (robot description, xacro)
@@ -14,8 +14,8 @@
         <gazebo reference="${prefix}lidar_link">
             <sensor name="${prefix}lidar_sensor" type="gpu_lidar">
-                <topic>/lidar</topic>
+                <topic>/scan</topic>
                 <update_rate>10</update_rate>
                 <always_on>true</always_on>
-                <visualize>true</visualize>
+                <visualize>false</visualize>
                 <lidar>
                     <scan>

File: mini_description/urdf/mini_common_materials.xacro (robot description, xacro)
@@ -8,5 +8,5 @@
     </material>
     <material name="white">
-        <color rgba="1.0 1.0 1.0 1.0"/>
+        <color rgba="1.0 1.0 1.0 0.3"/>
     </material>
 </robot>

File: mini_description/urdf/ros2_control/mini_ros2_control.xacro (robot description, xacro)
@@ -18,5 +18,5 @@
         <param name="timeout_ms">2000</param>
         <param name="enc_counts_per_rev">1062</param>
-        <param name="pid_p">160</param>
+        <param name="pid_p">200</param>
         <param name="pid_d">30</param>
         <param name="pid_i">15</param>

File: mini_description/urdf/sensors/mini_lidar.urdf.xacro (robot description, xacro)
@@ -1,10 +1,13 @@
 <?xml version="1.0"?>
 <robot xmlns:xacro="http://www.ros.org/wiki/xacro">
-    <xacro:property name="lidar_xoff" value="0.032966" />
+    <!-- <xacro:property name="lidar_xoff" value="0.032966" />
     <xacro:property name="lidar_yoff" value="0.0" />
-    <xacro:property name="lidar_zoff" value="0.083437" />
+    <xacro:property name="lidar_zoff" value="0.083437" /> -->
+    <xacro:property name="lidar_xoff" value="0.029" />
+    <xacro:property name="lidar_yoff" value="0.0" />
+    <xacro:property name="lidar_zoff" value="0.125" />
     <xacro:property name="lidar_mass" value="0.10321" />
-    <xacro:property name="lidar_length" value="0.043" />
-    <xacro:property name="lidar_width" value="0.04629" />
+    <xacro:property name="lidar_length" value="0.033" />
+    <xacro:property name="lidar_width" value="0.042" />
     <xacro:property name="lidar_height" value="0.0348" />
     <xacro:property name="com_x" value="-0.000082" />     <!--Center of Mass-->
@@ -12,4 +15,37 @@
     <xacro:property name="com_z" value="0.010541" />
     <xacro:macro name="mini_lidar" params="prefix">
+        <link name="${prefix}lidar_stand_link">
+            <visual>
+                <origin xyz="0.0 0.0 0.0" rpy="0.0 0.0 0.0"/>
+                <!-- <geometry>
+                    <mesh filename="file://$(find mini_description)/meshes/lidar.stl" scale="0.001 0.001 0.001"/>
+                </geometry> -->
+                <geometry>
+                    <box size="${lidar_length} ${lidar_width} 0.01"/>
+                </geometry>
+                <material name="white"/>
+            </visual>
+            <collision>
+                <origin xyz="0.0 0.0 0.0" rpy="0.0 0.0 0.0"/>
+                <!-- <geometry>
+                    <mesh filename="file://$(find mini_description)/meshes/lidar.stl" scale="0.001 0.001 0.001"/>
+                </geometry> -->
+                <geometry>
+                    <box size="${lidar_length} ${lidar_width} 0.01"/>
+                </geometry>
+            </collision>
+            <inertial>
+                <origin xyz="${com_x} ${com_y} ${com_z}" rpy="0 0 0"/>
+                <mass value="${lidar_mass*1.25}"/>
+                <inertia ixx="${(1/12) * lidar_mass * ((lidar_width * lidar_width) + (lidar_height * lidar_height))}"  ixy="0.0"  ixz="0.0"
+                            iyy="${(1/12) * lidar_mass * ((lidar_length * lidar_length) + (lidar_height * lidar_height))}"  iyz="0.0"
+                            izz="${(1/12) * lidar_mass * ((lidar_length * lidar_length) + (lidar_width * lidar_width))}"/>
+            </inertial>
+        </link>
+        <joint name="base_lidar_stand_joint" type="fixed">
+            <origin xyz="${lidar_xoff} ${lidar_yoff} ${lidar_zoff}" rpy="0.0 0.0 0.0"/>
+            <parent link="${prefix}base_link"/>
+            <child link="${prefix}lidar_stand_link"/>
+        </joint>
         <link name="${prefix}lidar_link">
             <visual>
@@ -34,7 +70,7 @@
         </link>
         <joint name="base_lidar_joint" type="fixed">
-            <origin xyz="${lidar_xoff} ${lidar_yoff} ${lidar_zoff}" rpy="0.0 0.0 0.0"/>
-            <parent link="base_link"/>
-            <child link="lidar_link"/>
+            <origin xyz="0 0 0.005" rpy="0.0 0.0 0.0"/>
+            <parent link="${prefix}lidar_stand_link"/>
+            <child link="${prefix}lidar_link"/>
         </joint>
     </xacro:macro>
